File: kicad_project/kicad_project.kicad_sch (KiCad schematic)
At the start: 22 parts, among them J1 USB_C_Receptacle_USB2.0_16P, Q1 DMG2302U, SW1 SW_Push, U1 STM32F031F6Px, U2 MCP73831-2-MC, U3 MCP4011-xxxxMS, U4 FT232RL, U5 LMZM23601

Commit message: first done
Parts:
- added C11: 10n, symbol Device:C
- added C12: 100n, symbol Device:C
- added FB1: FerriteBead, symbol Device:FerriteBead
- added R4: 470, symbol Device:R
Connections:
- net +3.3V: now also C9.1, U5.6 (VOUT), U5.7 (FB), C11.1, C12.1, FB1.2
- net +5V: now also C8.1, U5.3 (VIN), U5.4 (EN)
- net D+: now also J1.A6 (D+), J1.B6 (D+); no longer J1.A7 (D-), J1.B7 (D-)
- net D-: now also J1.A7 (D-), J1.B7 (D-); no longer J1.A6 (D+), J1.B6 (D+)
- net GND: now also C11.2, C12.2
- net at C5.1, U2.3 (V_{BAT}), U2.4 (V_{BAT}): now also Q1.2 (S)
- net adc_in7: now reaches Q1.3 (D)
- net adc_in7: now also U1.13 (PA7), R4.2
- net Cell+: now reaches U1.12 (PA6)
- net Cell+: now also U1.7 (PA1), R4.1
- net at U1.5 (VDDA): now also FB1.1
Other:
- moved on the sheet: C3, SW1

Commit message: temp modify
Parts:
- added C13: 10n, symbol Device:C
- added C14: 100n, symbol Device:C
Connections:
- net +3.3V: no longer C7.1, U4.17 (3V3OUT)
- net +5V: now also C13.1, C14.1
- net GND: now also C13.2, C14.2
- new net: C7.1, U4.17 (3V3OUT)
- no-connect marks 2 -> 16

Commit message: seg done
Parts:
- added Q2: DMG2302U, Package_TO_SOT_SMD:SOT-23, symbol Transistor_FET:DMG2302U
Connections:
- net +5V: now also Q2.2 (S); no longer C4.1, D1.2 (A), U2.1 (V_{DD}), U2.2 (V_{DD})
- net Cell+: now also C5.1, U2.3 (V_{BAT}), U2.4 (V_{BAT})
- net GND: now also C4.1, D1.2 (A), U2.1 (V_{DD}), U2.2 (V_{DD}), Q2.3 (D)
- net gate: now also Q2.1 (G)
- now unconnected: Q1.2 (S)
Other:
- moved on the sheet: C1, C11, C12, C2, C3, C4, C5, C6, C8, C9, D1, FB1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

Commit message: edit done
Parts:
- removed Q1: DMG2302U, Package_TO_SOT_SMD:SOT-23, symbol Transistor_FET:DMG2302U
- added R5: 220, symbol Device:R
- added R6: 10k, symbol Device:R
Connections:
- net +5V: now also Q2.3 (D); no longer Q2.2 (S)
- net Cell+: now also U1.14 (PB1); no longer U1.7 (PA1)
- net GND: now also Q2.2 (S), R6.2; no longer Q2.3 (D)
- net LED: now also U1.9 (PA3); no longer U1.20 (PA14)
- net gate: now also U1.7 (PA1), R5.1, R5.2, R6.1; no longer U1.19 (PA13)
- net stm_rx: now also U1.18 (PA10); no longer U1.9 (PA3)
- net stm_tx: now also U1.17 (PA9); no longer U1.8 (PA2)
- new net Buzzer: U1.8 (PA2)
- new net sys_swclk: U1.19 (PA13)
- new net sys_swdio: U1.20 (PA14)
Other:
- moved on the sheet: C10, J1, Q2, R2, R3

Commit message: edit done
Parts:
- removed C3: 100n, symbol Device:C
- removed SW1: SW_Push, symbol Switch:SW_Push
- added R7: 10k, symbol Device:R
Connections:
- net GND: now also R7.2
- net at U1.1 (BOOT0): now also R7.1
- no-connect marks 16 -> 17
Other:
- moved on the sheet: C1, C11, C12, C2, FB1, R4, U1

Commit message: edit done
Parts:
- removed R4: 470, symbol Device:R
- added BZ1: Buzzer, symbol Device:Buzzer
- added D2: LED, symbol Device:LED
- added R10: R_Shunt, symbol Device:R_Shunt
- added R8, R9: 10k, symbol Device:R
Connections:
- net Buzzer: now also R9.2
- net Cell+: now also R10.4; no longer C5.1, U1.12 (PA6), U2.3 (V_{BAT}), U2.4 (V_{BAT})
- net GND: now also BZ1.2 (-), D2.1 (K)
- net LED: now also R8.2
- net adc_in7: now also R10.2
- new net: D2.2 (A), R8.1
- new net: BZ1.1 (+), R9.1
- new net adc_in6: R10.3, U1.12 (PA6)
- new net charge ic: C5.1, R10.1, U2.3 (V_{BAT}), U2.4 (V_{BAT})

Commit message: edit done
Parts:
- added Q1: changeit, Package_TO_SOT_SMD:SOT-23, symbol Transistor_FET:DMG2302U
- added R4: 220, symbol Device:R
- added SW1: SW_DIP_x01, symbol Switch:SW_DIP_x01
- R10: value R_Shunt -> 0.01
- R9: value 10k -> 220
Connections:
- net +3.3V: now also SW1.1
- net +5V: now also Q1.3 (D)
- net GND: now also R4.2; no longer C4.1, D1.2 (A), Q2.2 (S), U2.1 (V_{DD}), U2.2 (V_{DD})
- net at R9.1: now also Q1.1 (G), R4.1; no longer BZ1.1 (+)
- net chg_prog: now reaches U2.8 (PROG), U3.3 (A)
- net at R7.1, U1.1 (BOOT0): now also SW1.2
- net stm_nrst: now reaches U1.4 (NRST)
- net Cell+ renamed BAT_monitor
- net adc_in6: no longer names the net of R10.3
- net adc_in6: no longer U1.12 (PA6)
- net adc_in7: no longer names the net of R10.2
- net adc_in7: no longer U1.13 (PA7)
- net charge ic: no longer names the net of C5.1, R10.1, U2.3 (V_{BAT}), U2.4 (V_{BAT})
- new net: C4.1, D1.2 (A), Q2.2 (S), U2.1 (V_{DD}), U2.2 (V_{DD})
- new net: BZ1.1 (+), Q1.2 (S)
- new net shunt: U1.12 (PA6)
- no-connect marks 17 -> 21
Other:
- moved on the sheet: BZ1, C1, C10, C11, C12, C2, C4, C5, C6, C7, C9, D1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
